Commit message: Able to rotate cube, and manipulate Z position using a gui slider, but no z transformation from the imu chip position.

File: install/imu_test/share/imu_test/urdf/robotmodel.urdf (robot description, URDF)
Before this commit: robot imu_test, 3 links, 2 joints
Joints:
- joint imu_dynamic_to_imu: axis (none) -> 0 0 1; limit (none) -> lower=-100.0 upper=100.0 effort=1000.0 velocity=10.0; type fixed -> prismatic

Commit message: Major push

File: install/imu_test/share/imu_test/urdf/robotmodel.urdf (robot description, URDF)
Before this commit: robot imu_test, 3 links, 2 joints
Links:
- removed link imu_link_dynamic
Joints:
- removed joint base_to_imu_dynamic
- removed joint imu_dynamic_to_imu
- added joint imu_joint: type prismatic, parent base_link, child imu_link, origin xyz=0 0 0 rpy=0 0 0, axis 0 0 1, limit lower=-1.0 upper=1.0 effort=1000.0 velocity=1.0
